File: opto.kicad_sch (KiCad schematic)
At the start: 18 parts, among them J5 UART_Device, U1 SN74LVC1G17DBVR, U10 TLP2361(TPL,E(T, U5 SN74LVC1G17DBVR, U8 SN74LVC1G17DBVR, U9 TLP2361(TPL,E(T

Commit message: eeschema wants this line gone.  Don't know why
Connections:
- net at U10.3: now also R23.1
Changed lines of the file:
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@@
 	)
 	(symbol
-		(lib_name "pypilot_components:tlp2361")
 		(lib_id "pypilot_components:tlp2361")
 		(at 182.88 40.64 0)

Commit message: Update all symbols
That it produced so little change confirms very little divergence from
stock and custom symbols.  Yippee!
Connections:
- net at U10.3: now also R23.1
Changed lines of the file:
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@@
 	)
 	(symbol
+		(lib_name "pypilot_components:tlp2361")
 		(lib_id "pypilot_components:tlp2361")
 		(at 182.88 40.64 0)
