File: clutch.kicad_sch (KiCad schematic)
At the start: 5 parts, among them J10 Clutch, Q6 SI2301

Commit message: Added results of fit test to components received from LCSC
Parts:
- J10: FitTest (none) -> Y
Changed lines of the file:
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@@
+			)
+		)
+		(property "FitTest" "Y"
+			(at 157.48 101.6 0)
+			(effects
+				(font
+					(size 1.27 1.27)
+				)
+				(hide yes)
 			)
 		)

Commit message: More fit test results
Parts:
- R27, R28: FitTest (none) -> Y
Changed lines of the file:
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@@
+			)
+		)
+		(property "FitTest" "Y"
+			(at 137.16 116.84 0)
+			(effects
+				(font
+					(size 1.27 1.27)
+				)
+				(hide yes)
 			)
 		)
@@
 			(effects
 				(font
+					(size 1.27 1.27)
+				)
+				(hide yes)
+			)
+		)
+		(property "FitTest" "Y"
+			(at 132.08 111.76 0)
+			(effects
+				(font
